File: Pikey/Pikey.kicad_sch (KiCad schematic)
At the start: 0 parts

Commit message: 11th April 2026 update
Parts:
- added C1, C2, C3, C7: 4.7u, Capacitor_SMD:C_0402_1005Metric, symbol Device:C
- added C10, C11, C12, C13, C14, C15, C16, C17, C18, C6, C8, C9: 100u, Capacitor_SMD:C_0402_1005Metric, symbol Device:C
- added C19, C20: 15p, Capacitor_SMD:C_0402_1005Metric, symbol Device:C
- added C4, C5: 10u, Capacitor_SMD:C_0402_1005Metric, symbol Device:C
- added D1, D10, D11, D12, D13, D14, D15, D16, D2, D3, D4, D5, D6, D7, D8, D9: SK6812, LED_SMD:LED_SK6812_PLCC4_5.0x5.0mm_P3.2mm, symbol LED:SK6812
- added D17, D18: D, Diode_SMD:D_0402_1005Metric, symbol Device:D
- added D19: SMLVN6RGB, LED_SMD:LED_2010_5025Metric, symbol LED:SMLVN6RGB
- added J1: DX07P024AJ1R1500, DX07P024AJ1R1500:JAE_DX07P024AJ1R1500, symbol DX07P024AJ1R1500:DX07P024AJ1R1500
- added J2: Conn_01x03, Connector_PinHeader_1.00mm:PinHeader_1x03_P1.00mm_Vertical_SMD, symbol Connector_Generic:Conn_01x03
- added L2: AOTA-B201610S3R3-101-T, AOTAB201610S3R3101T, symbol AOTA-B201610S3R3-101-T:AOTA-B201610S3R3-101-T
- added R1: 5.1k, Resistor_SMD:R_0201_0603Metric, symbol Device:R
- added R2, R3: 27, Resistor_SMD:R_0201_0603Metric, symbol Device:R
- added R4: 33, Resistor_SMD:R_0402_1005Metric, symbol Device:R
- added R5, R6: 1k, Resistor_SMD:R_0402_1005Metric, symbol Device:R
- added R7: 9.1kΩ, Resistor_SMD:R_0201_0603Metric, symbol Device:R
- added R8: 6.2kΩ, Resistor_SMD:R_0201_0603Metric, symbol Device:R
- added S1: SKRPACE010, SKRPACE010:SW_SKRPACE010, symbol SKRPACE010:SKRPACE010
- added SW1, SW2: CK_KMS2xxG, Button_Switch_SMD:SW_SPST_CK_KMS2xxGP, symbol Switch:CK_KMS2xxG
- added U1: RP2350B, Package_DFN_QFN:QFN-80-1EP_10x10mm_P0.4mm_EP3.4x3.4mm, symbol MCU_RaspberryPi:RP2350B
- added U2: NCP1117-3.3_SOT223, Package_TO_SOT_SMD:SOT-223-3_TabPin2, symbol Regulator_Linear:NCP1117-3.3_SOT223
- added U3: W25Q128JVS, Package_SO:SOIC-8_5.3x5.3mm_P1.27mm, symbol Memory_Flash:W25Q128JVS
- added Y1: ABM8-272-T3, ABM8-272-T3:XTAL_ABM8-272-T3, symbol ABM8-272-T3:ABM8-272-T3
Connections:
- new net: D11.4 (DOUT), D12.2 (DIN)
- new net: D12.4 (DOUT), D13.2 (DIN)
- new net: C10.1, C11.1, C12.1, C13.1, C14.1, C15.1, C16.1, C17.1, C9.1, U1.15 (IOVDD), U1.24 (IOVDD), U1.29 (IOVDD), U1.41 (IOVDD), U1.5 (IOVDD), U1.50 (IOVDD), U1.59 (ADC_AVDD), U1.60 (IOVDD), U1.68 (USB_OTP_VDD), U1.69 (QSPI_IOVDD), U1.76 (IOVDD)
- new net: C1.2, R4.1, U1.61 (VREG_AVDD)
- new net: D1.2 (DIN), D4.4 (DOUT)
- new net: D1.4 (DOUT), D2.2 (DIN)
- new net: SW2.1, U1.35 (RUN)
- new net: D5.4 (DOUT), D6.2 (DIN)
- new net: D6.4 (DOUT), D7.2 (DIN)
- new net: J2.1 (Pin_1), U1.34 (SWDIO)
- new net: J2.3 (Pin_3), U1.33 (SWCLK)
- new net: D19.1 (BA), S1.3
- new net: D19.2 (RA), U1.78 (GPIO1)
- new net: D19.3 (GA), U1.79 (GPIO2)
- new net: J1.A5 (CC), R1.2
- new net: J1.A6 (D+), R2.2
- new net: J1.A7 (D-), R3.2
- new net: C20.2, R6.1, U1.31 (XOUT)
- new net: R6.2, Y1.1
- new net: D15.4 (DOUT), D16.2 (DIN)
- new net: D2.4 (DOUT), D3.2 (DIN)
- new net: L2.1, U1.63 (VREG_LX)
- new net: C19.2, U1.30 (XIN), Y1.3
- new net: D10.4 (DOUT), D11.2 (DIN)
- new net: R5.2, SW1.1
- new net: R7.1, R8.1
- new net: R7.2, S1.4
- new net: D13.4 (DOUT), D14.2 (DIN)
- new net: D3.4 (DOUT), D5.2 (DIN)
- new net: D10.2 (DIN), D9.4 (DOUT)
- new net: S1.2, U1.77 (GPIO0)
- new net: D14.4 (DOUT), D15.2 (DIN)
- new net: R5.1, U1.75 (~{QSPI_SS}), U3.1 (~{CS})
- new net: U1.74 (QSPI_SD1), U3.2 (DO/IO_{1})
- new net: U1.73 (QSPI_SD2), U3.3 (~{WP}/IO_{2})
- new net: U1.72 (QSPI_SD0), U3.5 (DI/IO_{0})
- new net: U1.71 (QSPI_SCLK), U3.6 (CLK)
- new net: U1.70 (QSPI_SD3), U3.7 (~{HOLD}/~{RESET}/IO_{3})
- new net: D7.4 (DOUT), D8.2 (DIN)
- new net: D8.4 (DOUT), D9.2 (DIN)
- new net +3.3V: C18.1, C2.1, C5.2, R4.2, R8.2, U1.64 (VREG_VIN), U2.2 (VO), U3.8 (VCC)
- new net +5V: C4.2, D17.1 (K), D18.1 (K), U2.3 (VI)
- new net 1.1V: C3.1, C6.1, C7.1, C8.1, L2.2, U1.10 (DVDD), U1.32 (DVDD), U1.51 (DVDD), U1.65 (VREG_FB)
- new net DM: R2.1, U1.66 (USB_DM)
- new net DP: R3.1, U1.67 (USB_DP)
- new net GND: C1.1, C10.2, C11.2, C12.2, C13.2, C14.2, C15.2, C16.2, C17.2, C18.2, C19.1, C2.2, C20.1, C3.2, C4.1, C5.1, C6.2, C7.2, C8.2, C9.2, D19.4 (GK), D19.5 (RK), D19.6 (BK), J1.A1 (GND_A), J1.A12 (GND_A), J1.B1 (GND_B), J1.B12 (GND_B), J1.S3 (SHIELD), J1.S4 (SHIELD), J1.S5 (SHIELD), J1.S6 (SHIELD), J2.2 (Pin_2), R1.1, S1.1, SW1.2, SW1.SH (B), SW2.2, SW2.SH (B), U1.62 (VREG_PGND), U1.81 (GND), U2.1 (GND), U3.4 (GND), Y1.2 (GND), Y1.4 (GND)
- new net VBUS_A: D17.2 (A), J1.A4 (VBUS_A), J1.A9 (VBUS_A)
- new net VBUS_B: D18.2 (A), J1.B4 (VBUS_B), J1.B9 (VBUS_B)
