File: Pikey/Pikey.kicad_sch (KiCad schematic)
At the start: 58 parts, among them J1 DX07P024AJ1R1500, J2 Conn_01x03, J3 Micro_SD_Card_Det2, SW1 CK_KMS2xxG, SW2 CK_KMS2xxG, U1 RP2350B, U2 NCP1117-3.3_SOT223, U3 W25Q128JVS, Y1 ABM8-272-T3

Commit message: 13th April update
added the nRF8001
Parts:
- added C21, C23, C25, C29: 10uF, Capacitor_SMD:C_0402_1005Metric, symbol Device:C
- added C22, C24, C26, C27, C28: 100nF, Capacitor_SMD:C_0402_1005Metric, symbol Device:C
- added FB1, FB2, FB3: FerriteBead, Inductor_SMD:L_0402_1005Metric, symbol Device:FerriteBead
- added R10, R11, R12, R13, R9: 10k, Resistor_SMD:R_0201_0603Metric, symbol Device:R
- added U4: nRF8001, Package_DFN_QFN:QFN-32-1EP_5x5mm_P0.5mm_EP3.45x3.45mm, symbol RF_Bluetooth:nRF8001
Connections:
- net +3.3V: now also J3.4 (VDD), C27.1, C28.1, C29.1, FB1.1, FB2.1, FB3.1, R10.2, R11.2, R12.2, R13.2, R9.2, U4.1 (VDD), U4.9 (VDD)
- net GND: now also J3.10 (DET_A), J3.9 (DET_B), U1.42 (GPIO33), C22.2, C24.2, C26.2, C27.2, C28.2, C29.2, U4.17 (VSS), U4.18 (VSS), U4.23 (VSS), U4.30 (VSS), U4.31 (VSS), U4.8 (VSS)
- net DAT2: now reaches J3.1 (DAT2)
- net DAT2: now also U1.47 (GPIO38), R9.1
- net DAT3: now reaches J3.2 (DAT3/CD)
- net DAT3: now also U1.48 (GPIO39), R10.1
- net CMD: now reaches J3.3 (CMD)
- net CMD: now also U1.43 (GPIO34), R11.1
- net CLK: now reaches J3.5 (CLK)
- net CLK: now also U1.44 (GPIO35)
- net DAT0: now reaches J3.7 (DAT0)
- net DAT0: now also U1.45 (GPIO36), R12.1
- net DAT1: now reaches J3.8 (DAT1)
- net DAT1: now also U1.46 (GPIO37), R13.1
- new net: C21.1, FB3.2, U4.24 (AVDD)
- new net: C21.2, C22.1
- new net: C23.2, C24.1
- new net: C25.2, C26.1
- new net: C25.1, FB2.2, U4.29 (AVDD)
- new net: C23.1, FB1.2, U4.26 (AVDD)

Commit message: updateee
Parts:
- removed D1, D10, D11, D12, D13, D14, D15, D16, D2, D3, D4, D5, D6, D7, D8, D9: SK6812, LED_SMD:LED_SK6812_PLCC4_5.0x5.0mm_P3.2mm, symbol LED:SK6812
- added C30, C31: 100nF, Capacitor_SMD:C_0402_1005Metric, symbol Device:C
- added C32, C33: 10pF, Capacitor_SMD:C_0402_1005Metric, symbol Device:C
- added E1: ANT3216A063R2400A, ANT3216A063R2400A:XDCR_ANT3216A063R2400A, symbol ANT3216A063R2400A:ANT3216A063R2400A
- added U5: BAL-NRF01D3, BAL-NRF01D3:IC_BAL-NRF01D3, symbol BAL-NRF01D3:BAL-NRF01D3
- added Y2: ABS05-32.768KHZ-T, ABS05-32.768KHZ-T:XTAL_ABS05-32.768KHZ-T, symbol ABS05-32.768KHZ-T:ABS05-32.768KHZ-T
- added Y3: ABM8-16.000MHZ-B2-T, ABM8-16.000MHZ-B2-T:XTAL_ABM8-16.000MHZ-B2-T, symbol ABM8-16.000MHZ-B2-T:ABM8-16.000MHZ-B2-T
- C1, C2, C3, C7: value 4.7u -> 4.7uF; LCSC Part number (none) -> C23733; Name (none) -> Samsung Electro-Mechanics CL05A475MP5NRNC
- C10, C11, C12, C13, C14, C15, C16, C17, C18, C6, C8, C9: value 100u -> 100uF; LCSC Part number (none) -> C26409; Name (none) -> Samsung Electro-Mechanics CL05C101JB5NNNC
- C19, C20: value 15p -> 15pF; LCSC Part number (none) -> C86285; Name (none) -> Samsung Electro-Mechanics CL05C150JB5NNNC
- C21, C23, C25, C29: LCSC Part number (none) -> C315248; Name (none) -> Samsung Electro-Mechanics CL05A106MP5NUNC
- C22, C24, C26, C27, C28: LCSC Part number (none) -> C1525; Name (none) -> Samsung Electro-Mechanics CL05B104KO5NNNC
- C4, C5: value 10u -> 10uF; LCSC Part number (none) -> C315248; Name (none) -> Samsung Electro-Mechanics CL05A106MP5NUNC
- D17, D18: value D -> 5V; LCSC Part number (none) -> C145179; Name (none) -> onsemi RB521S30T1G
- D19: LCSC Part number (none) -> C2842809; Name (none) -> ROHM SMLVN6RGB1W1
- FB1, FB2, FB3: LCSC Part number (none) -> C19330; Name (none) -> muRata BLM18AG601SN1D
- J1: LCSC Part number (none) -> C5352764; Name (none) -> JAE Electronics DX07P024AJ1R1500
- J2: now left out of the parts list
- J3: value Micro_SD_Card_Det2 -> Microsd card; LCSC Part number (none) -> C114218; Name (none) -> HRS DM3AT-SF-PEJM5
- L2: LCSC Part number (none) -> C42411119; Name (none) -> ABRACON AOTA-B201610S3R3-101-T
- R1: value 5.1k -> 5.1kΩ; LCSC Part number (none) -> C105872; Name (none) -> YAGEO RC0402FR-075K1L
- R10, R11, R12, R13, R9: value 10k -> 10kΩ; LCSC Part number (none) -> C60490; Name (none) -> YAGEO RC0402FR-0710KL
- R2, R3: value 27 -> 27Ω; LCSC Part number (none) -> C413051; Name (none) -> PANASONIC ERJ2RKF27R0X
- R4: value 33 -> 33Ω; LCSC Part number (none) -> C2906868; Name (none) -> FOJAN FRC0402F33R0TS
- R5, R6: value 1k -> 1kΩ; LCSC Part number (none) -> C106235; Name (none) -> YAGEO RC0402FR-071KL
- R7: LCSC Part number (none) -> C163450; Name (none) -> YAGEO RC0402FR-079K1L
- R8: LCSC Part number (none) -> C137946; Name (none) -> YAGEO RC0402FR-076K2L
- S1: LCSC Part number (none) -> C139797; Name (none) -> ALPSALPINE SKRPACE010
- SW1, SW2: LCSC Part number (none) -> C221701; Name (none) -> C&K KMS231GLFS
- U1: LCSC Part number (none) -> C42415655; Name (none) -> Raspberry Pi RP2350B
- U2: LCSC Part number (none) -> C26537; Name (none) -> onsemi NCP1117ST33T3G
- U3: LCSC Part number (none) -> C97521; Name (none) -> Winbond W25Q128JVSIQ
- U4: LCSC Part number (none) -> C5200800; Name (none) -> NORDIC nRF8001-R2Q32-R
- Y1: LCSC Part number (none) -> C20625731; Name (none) -> ABRACON ABM8-272-T3
Connections:
- net +3.3V: now also U5.C2 (VCC)
- net GND: now also C30.2, C31.2, C32.2, C33.2, E1.S1_2, E1.S2, U5.A2 (GND), Y3.2 (GND), Y3.4 (GND)
- net GPIO10: now reaches U4.11 (SCK)
- net GPIO10: now also U1.8 (GPIO10)
- net GPIO13: now reaches U4.12 (REQN)
- net GPIO13: now also U1.12 (GPIO13)
- net GPIO12: now reaches U4.13 (MOSI)
- net GPIO12: now also U1.11 (GPIO12)
- net GPIO11: now reaches U4.14 (MISO)
- net GPIO11: now also U1.9 (GPIO11)
- net GPIO14: now reaches U4.16 (RDYN)
- net GPIO14: now also U1.13 (GPIO14)
- net GPIO15: now reaches U4.19 (RESET)
- net GPIO15: now also U1.14 (GPIO15)
- net at U4.2 (DEC1): now also C30.1
- net at U4.21 (ANT1): now also U5.C3 (DIFF2)
- net at U4.22 (ANT2): now also U5.A3 (DIFF1)
- net at U4.27 (XC2): now also Y3.3
- net at U4.28 (XC1): now also Y3.1
- net at U4.3 (DEC2): now also C31.1
- net at U4.4 (XL2): now also U4.5 (XL1), U4.6 (ACTIVE), C32.1, C33.1, Y2.1, Y2.2
- new net: E1.S1_1, U5.B1 (SE)
Other:
- moved on the sheet: C4, C5

Commit message: 20th april update
Parts:
- removed C21, C23, C25: 10uF, Capacitor_SMD:C_0402_1005Metric, symbol Device:C
- removed C22, C24, C26, C27, C28, C30, C31: 100nF, Capacitor_SMD:C_0402_1005Metric, symbol Device:C
- removed C32, C33: 10pF, Capacitor_SMD:C_0402_1005Metric, symbol Device:C
- removed E1: ANT3216A063R2400A, ANT3216A063R2400A:XDCR_ANT3216A063R2400A, symbol ANT3216A063R2400A:ANT3216A063R2400A
- removed FB1, FB2, FB3: FerriteBead, Inductor_SMD:L_0402_1005Metric, symbol Device:FerriteBead
- removed U4: nRF8001, Package_DFN_QFN:QFN-32-1EP_5x5mm_P0.5mm_EP3.45x3.45mm, symbol RF_Bluetooth:nRF8001
- removed U5: BAL-NRF01D3, BAL-NRF01D3:IC_BAL-NRF01D3, symbol BAL-NRF01D3:BAL-NRF01D3
- removed Y2: ABS05-32.768KHZ-T, ABS05-32.768KHZ-T:XTAL_ABS05-32.768KHZ-T, symbol ABS05-32.768KHZ-T:ABS05-32.768KHZ-T
- removed Y3: ABM8-16.000MHZ-B2-T, ABM8-16.000MHZ-B2-T:XTAL_ABM8-16.000MHZ-B2-T, symbol ABM8-16.000MHZ-B2-T:ABM8-16.000MHZ-B2-T
Other:
- moved on the sheet: C29, J3, R10, R11, R12, R13, R9

Commit message: May 2nd update
Parts:
- removed D19: SMLVN6RGB, LED_SMD:LED_2010_5025Metric, symbol LED:SMLVN6RGB
- removed J1: DX07P024AJ1R1500, DX07P024AJ1R1500:JAE_DX07P024AJ1R1500, symbol DX07P024AJ1R1500:DX07P024AJ1R1500
- removed SW1, SW2: CK_KMS2xxG, Button_Switch_SMD:SW_SPST_CK_KMS2xxGP, symbol Switch:CK_KMS2xxG
- added D1: SMLVN6RGB, LED_SMD:LED_ROHM_SMLVN6, symbol LED:SMLVN6RGB
- added J1, J5: Conn_02x01, Connector_PinHeader_1.00mm:PinHeader_2x01_P1.00mm_Vertical, symbol Connector_Generic:Conn_02x01
- added J2: DX07P024MJ1R1500, DX07P024MJ1R1500:JAE_DX07P024MJ1R1500, symbol DX07P024MJ1R1500:DX07P024MJ1R1500
- added R14: 5.1kΩ, Resistor_SMD:R_0201_0603Metric, symbol Device:R
- J4: renamed from J2; footprint Connector_PinHeader_1.00mm:PinHeader_1x03_P1.00mm_Vertical_SMD -> Connector_PinHeader_1.00mm:PinHeader_1x03_P1.00mm_Vertical
- L2: footprint AOTAB201610S3R3101T -> AOTA-B201610S3R3-101-T:AOTAB201610S3R3101T
Connections:
- net GND: now also D1.4 (GK), D1.5 (RK), D1.6 (BK), J1.2 (Pin_2), J2.A1 (GNDA), J2.A12 (GNDA), J2.B1 (GNDB), J2.B12 (GNDB), J2.S3 (SHIELD), J2.S4 (SHIELD), J2.S5 (SHIELD), J2.S6 (SHIELD), J5.2 (Pin_2), R14.1
- net at U1.35 (RUN): now also J5.1 (Pin_1)
- net at S1.3: now also D1.1 (BA)
- net at U1.78 (GPIO1): now also D1.2 (RA)
- net at U1.79 (GPIO2): now also D1.3 (GA)
- net at R1.2: now also J2.A5 (CC1)
- net at R2.2: now also J2.A7 (DA-), J2.B7 (DB-)
- net at R3.2: now also J2.A6 (DA+), J2.B6 (DB+)
- net at R5.2: now also J1.1 (Pin_1)
- net VBUS_A renamed A_VBUS
- net A_VBUS: now also J2.A4 (A_VBUS), J2.A9 (A_VBUS)
- net VBUS_B renamed B_VBUS
- net B_VBUS: now also J2.B4 (B_VBUS), J2.B9 (B_VBUS)
- new net: J2.B5 (CC2), R14.2

Commit message: Monday 4th May update
Parts:
- D1: LCSC Part number (none) -> C2909770; Name (none) -> ROHM SMLVN6RGB1U1
- J1, J5: now left out of the parts list
- J2: LCSC Part number (none) -> C134112; Name (none) -> JAE Electronics DX07P024MJ1R1500
Connections:
- net CLK: now also U1.19 (GPIO19); no longer U1.44 (GPIO35)
- net CMD: now also U1.18 (GPIO18); no longer J3.3 (CMD), R11.1, U1.43 (GPIO34)
- net DAT0: now also U1.20 (GPIO20); no longer U1.45 (GPIO36)
- net DAT1: now also U1.21 (GPIO21); no longer U1.46 (GPIO37)
- net DAT2: now also U1.22 (GPIO22); no longer U1.47 (GPIO38)
- net DAT3: now also U1.23 (GPIO23); no longer U1.48 (GPIO39)
- net GND: now also U1.17 (GPIO17); no longer U1.42 (GPIO33)
- new net: J3.3 (CMD), R11.1
Other:
- moved on the sheet: R10, R11, R9
