File: Pikey/Pikey.kicad_pcb (KiCad board)
At the start: 2 copper layers, 18 parts, among them U1 RP2350B

Commit message: 20th april update
Parts:
- removed D1, D10, D11, D12, D13, D14, D15, D16, D2, D3, D4, D5, D6, D7, D8, D9: SK6812, LED_SMD:LED_SK6812_PLCC4_5.0x5.0mm_P3.2mm
- removed REF**: PinHeader_1x03_P1.00mm_Vertical_SMD, Connector_PinHeader_1.00mm:PinHeader_1x03_P1.00mm_Vertical_SMD
- added C1: 4.7uF, Capacitor_SMD:C_0402_1005Metric, F.Cu at (73.2, 72.8)
- added C10: 100uF, Capacitor_SMD:C_0402_1005Metric, F.Cu at (76.0, 76.8)
- added C11: 100uF, Capacitor_SMD:C_0402_1005Metric, F.Cu at (76.0, 78.7)
- added C12: 100uF, Capacitor_SMD:C_0402_1005Metric, F.Cu at (76.0, 80.7)
- added C13: 100uF, Capacitor_SMD:C_0402_1005Metric, F.Cu at (76.0, 82.7)
- added C14: 100uF, Capacitor_SMD:C_0402_1005Metric, F.Cu at (76.0, 84.7)
- added C15: 100uF, Capacitor_SMD:C_0402_1005Metric, F.Cu at (78.9, 72.8)
- added C16: 100uF, Capacitor_SMD:C_0402_1005Metric, F.Cu at (78.9, 74.8)
- added C17: 100uF, Capacitor_SMD:C_0402_1005Metric, F.Cu at (78.9, 76.8)
- added C18: 100uF, Capacitor_SMD:C_0402_1005Metric, F.Cu at (78.9, 78.7)
- added C19: 15pF, Capacitor_SMD:C_0402_1005Metric, F.Cu at (78.9, 80.7)
- added C2: 4.7uF, Capacitor_SMD:C_0402_1005Metric, F.Cu at (73.2, 74.8)
- added C20: 15pF, Capacitor_SMD:C_0402_1005Metric, F.Cu at (78.9, 82.7)
- added C29: 10uF, Capacitor_SMD:C_0402_1005Metric, F.Cu at (84.7, 72.8)
- added C3: 4.7uF, Capacitor_SMD:C_0402_1005Metric, F.Cu at (73.2, 76.8)
- added C4: 10uF, Capacitor_SMD:C_0402_1005Metric, F.Cu at (73.2, 78.7)
- added C5: 10uF, Capacitor_SMD:C_0402_1005Metric, F.Cu at (73.2, 80.7)
- added C6: 100uF, Capacitor_SMD:C_0402_1005Metric, F.Cu at (73.2, 82.7)
- added C7: 4.7uF, Capacitor_SMD:C_0402_1005Metric, F.Cu at (73.2, 84.7)
- added C8: 100uF, Capacitor_SMD:C_0402_1005Metric, F.Cu at (76.0, 72.8)
- added C9: 100uF, Capacitor_SMD:C_0402_1005Metric, F.Cu at (76.0, 74.8)
- added D17: 5V, Diode_SMD:D_0402_1005Metric, F.Cu at (92.7, 89.8)
- added D18: 5V, Diode_SMD:D_0402_1005Metric, F.Cu at (92.7, 91.8)
- added D19: SMLVN6RGB, LED_SMD:LED_2010_5025Metric, F.Cu at (58.7, 89.6)
- added J1: DX07P024AJ1R1500, DX07P024AJ1R1500:JAE_DX07P024AJ1R1500, F.Cu at (118.2, 61.2)
- added J2: Conn_01x03, Connector_PinHeader_1.00mm:PinHeader_1x03_P1.00mm_Vertical_SMD, F.Cu at (92.7, 85.3)
- added J3: Microsd card, Connector_Card:microSD_HC_Hirose_DM3AT-SF-PEJM5, F.Cu at (117.8, 89.7)
- added L2: AOTA-B201610S3R3-101-T, AOTA-B201610S3R3-101-T:AOTAB201610S3R3101T, F.Cu at (65.7, 87.2)
- added R1: 5.1kΩ, Resistor_SMD:R_0201_0603Metric, F.Cu at (87.3, 84.7)
- added R10: 10kΩ, Resistor_SMD:R_0201_0603Metric, F.Cu at (89.8, 86.4)
- added R11: 10kΩ, Resistor_SMD:R_0201_0603Metric, F.Cu at (89.8, 88.2)
- added R12: 10kΩ, Resistor_SMD:R_0201_0603Metric, F.Cu at (89.8, 89.9)
- added R13: 10kΩ, Resistor_SMD:R_0201_0603Metric, F.Cu at (89.8, 91.7)
- added R2: 27Ω, Resistor_SMD:R_0201_0603Metric, F.Cu at (87.3, 86.4)
- added R3: 27Ω, Resistor_SMD:R_0201_0603Metric, F.Cu at (87.3, 88.2)
- added R4: 33Ω, Resistor_SMD:R_0402_1005Metric, F.Cu at (87.5, 78.8)
- added R5: 1kΩ, Resistor_SMD:R_0402_1005Metric, F.Cu at (87.5, 80.8)
- added R6: 1kΩ, Resistor_SMD:R_0402_1005Metric, F.Cu at (87.5, 82.8)
- added R7: 9.1kΩ, Resistor_SMD:R_0201_0603Metric, F.Cu at (87.3, 89.9)
- added R8: 6.2kΩ, Resistor_SMD:R_0201_0603Metric, F.Cu at (87.3, 91.7)
- added R9: 10kΩ, Resistor_SMD:R_0201_0603Metric, F.Cu at (89.8, 84.7)
- added S1: SKRPACE010, SKRPACE010:SW_SKRPACE010, F.Cu at (66.2, 82.5)
- added SW1: CK_KMS2xxG, Button_Switch_SMD:SW_SPST_CK_KMS2xxGP, F.Cu at (92.3, 74.3)
- added SW2: CK_KMS2xxG, Button_Switch_SMD:SW_SPST_CK_KMS2xxGP, F.Cu at (92.3, 79.7)
- added U2: NCP1117-3.3_SOT223, Package_TO_SOT_SMD:SOT-223-3_TabPin2, F.Cu at (95.9, 76.2)
- added U3: W25Q128JVS, Package_SO:SOIC-8_5.3x5.3mm_P1.27mm, F.Cu at (76.9, 89.2)
- added Y1: ABM8-272-T3, ABM8-272-T3:XTAL_ABM8-272-T3, F.Cu at (92.1, 67.4)
- moved U1 30.5 mm to (118.2, 73.3)
Connections:
- U1 pad 10: Net-(U1-DVDD-Pad10) -> 1.1V
- U1 pad 11: unconnected-(U1-GPIO12-Pad11) -> GPIO12
- U1 pad 12: unconnected-(U1-GPIO13-Pad12) -> GPIO13
- U1 pad 13: unconnected-(U1-GPIO14-Pad13) -> GPIO14
- U1 pad 14: unconnected-(U1-GPIO15-Pad14) -> GPIO15
- U1 pad 15: Net-(U1-IOVDD-Pad15) -> Net-(U1-ADC_AVDD)
- U1 pad 24: Net-(U1-IOVDD-Pad15) -> Net-(U1-ADC_AVDD)
- U1 pad 29: Net-(U1-IOVDD-Pad15) -> Net-(U1-ADC_AVDD)
- U1 pad 30: unconnected-(U1-XIN-Pad30) -> Net-(U1-XIN)
- U1 pad 31: unconnected-(U1-XOUT-Pad31) -> Net-(U1-XOUT)
- U1 pad 32: Net-(U1-DVDD-Pad10) -> 1.1V
- U1 pad 33: unconnected-(U1-SWCLK-Pad33) -> Net-(J2-Pin_3)
- U1 pad 34: unconnected-(U1-SWDIO-Pad34) -> Net-(J2-Pin_1)
- U1 pad 35: unconnected-(U1-RUN-Pad35) -> Net-(U1-RUN)
- U1 pad 41: Net-(U1-IOVDD-Pad15) -> Net-(U1-ADC_AVDD)
- U1 pad 42: unconnected-(U1-GPIO33-Pad42) -> DET
- U1 pad 43: unconnected-(U1-GPIO34-Pad43) -> CMD
- U1 pad 44: unconnected-(U1-GPIO35-Pad44) -> CLK
- U1 pad 45: unconnected-(U1-GPIO36-Pad45) -> DAT0
- U1 pad 46: unconnected-(U1-GPIO37-Pad46) -> DAT1
- U1 pad 47: unconnected-(U1-GPIO38-Pad47) -> DAT2
- U1 pad 48: unconnected-(U1-GPIO39-Pad48) -> DAT3
- U1 pad 5: Net-(U1-IOVDD-Pad15) -> Net-(U1-ADC_AVDD)
- U1 pad 50: Net-(U1-IOVDD-Pad15) -> Net-(U1-ADC_AVDD)
- U1 pad 51: Net-(U1-DVDD-Pad10) -> 1.1V
- U1 pad 59: unconnected-(U1-ADC_AVDD-Pad59) -> Net-(U1-ADC_AVDD)
- U1 pad 60: Net-(U1-IOVDD-Pad15) -> Net-(U1-ADC_AVDD)
- U1 pad 61: unconnected-(U1-VREG_AVDD-Pad61) -> Net-(U1-VREG_AVDD)
- U1 pad 62: unconnected-(U1-VREG_PGND-Pad62) -> DET
- U1 pad 63: unconnected-(U1-VREG_LX-Pad63) -> Net-(U1-VREG_LX)
- U1 pad 64: unconnected-(U1-VREG_VIN-Pad64) -> +3.3V
- U1 pad 65: unconnected-(U1-VREG_FB-Pad65) -> 1.1V
- U1 pad 66: unconnected-(U1-USB_DM-Pad66) -> DM
- U1 pad 67: unconnected-(U1-USB_DP-Pad67) -> DP
- U1 pad 68: unconnected-(U1-USB_OTP_VDD-Pad68) -> Net-(U1-ADC_AVDD)
- U1 pad 69: unconnected-(U1-QSPI_IOVDD-Pad69) -> Net-(U1-ADC_AVDD)
- U1 pad 70: unconnected-(U1-QSPI_SD3-Pad70) -> Net-(U1-QSPI_SD3)
- U1 pad 71: unconnected-(U1-QSPI_SCLK-Pad71) -> Net-(U1-QSPI_SCLK)
- U1 pad 72: unconnected-(U1-QSPI_SD0-Pad72) -> Net-(U1-QSPI_SD0)
- U1 pad 73: unconnected-(U1-QSPI_SD2-Pad73) -> Net-(U1-QSPI_SD2)
- U1 pad 74: unconnected-(U1-QSPI_SD1-Pad74) -> Net-(U1-QSPI_SD1)
- U1 pad 75: unconnected-(U1-~{QSPI_SS}-Pad75) -> Net-(U1-~{QSPI_SS})
- U1 pad 76: Net-(U1-IOVDD-Pad15) -> Net-(U1-ADC_AVDD)
- U1 pad 77: unconnected-(U1-GPIO0-Pad77) -> Net-(U1-GPIO0)
- U1 pad 78: unconnected-(U1-GPIO1-Pad78) -> Net-(D19-RA)
- U1 pad 79: unconnected-(U1-GPIO2-Pad79) -> Net-(D19-GA)
- U1 pad 8: unconnected-(U1-GPIO10-Pad8) -> GPIO10
- U1 pad 81: unconnected-(U1-GND-Pad81) -> DET
- U1 pad 9: unconnected-(U1-GPIO11-Pad9) -> GPIO11
Other:
- board outline added: 8.4 x 4.1 mm

Commit message: May 2nd update
Parts:
- removed D19: SMLVN6RGB, LED_SMD:LED_2010_5025Metric
- removed SW1, SW2: CK_KMS2xxG, Button_Switch_SMD:SW_SPST_CK_KMS2xxGP
- added D1: SMLVN6RGB, LED_SMD:LED_ROHM_SMLVN6, F.Cu at (115.5, 54.7)
- added J4: Conn_01x03, Connector_PinHeader_1.00mm:PinHeader_1x03_P1.00mm_Vertical, B.Cu at (111.7, 54.6)
- added J5: Conn_02x01, Connector_PinHeader_1.00mm:PinHeader_2x01_P1.00mm_Vertical, F.Cu at (125.3, 67.2)
- added R14: 5.1kΩ, Resistor_SMD:R_0201_0603Metric, F.Cu at (124.5, 59.7)
- C1, C10, C11, C12, C13, C14, C15, C16, C17, C18, C19, C2, C20, C29, C3, C4, C5, C6, C7, C8, C9, L2, R1, R10, R11, R12, R13, R2, R3, R4, R5, R6, R7, R8, R9, U2, U3, Y1: moved to B.Cu
- J1: value DX07P024AJ1R1500 -> Conn_02x01; footprint DX07P024AJ1R1500:JAE_DX07P024AJ1R1500 -> Connector_PinHeader_1.00mm:PinHeader_2x01_P1.00mm_Vertical
- J2: value Conn_01x03 -> DX07P024MJ1R1500; footprint Connector_PinHeader_1.00mm:PinHeader_1x03_P1.00mm_Vertical_SMD -> DX07P024MJ1R1500:JAE_DX07P024MJ1R1500
- moved L2 61.8 mm to (123.4, 64.9), turned to -90 degrees
- moved S1 61.4 mm to (121.0, 54.7)
- moved C5 50.7 mm to (123.8, 77.5), turned to 90 degrees
- moved C6 49.9 mm to (122.8, 77.5), turned to 90 degrees
- moved C7 49.2 mm to (121.9, 77.5), turned to 90 degrees
- moved C12 48.0 mm to (123.8, 75.6), turned to 90 degrees
- moved C13 47.3 mm to (122.8, 75.6), turned to 90 degrees
- moved J2 46.8 mm to (118.4, 46.2), turned to 180 degrees
- moved C14 46.7 mm to (121.9, 75.6), turned to 90 degrees
- moved C4 46.2 mm to (119.3, 77.9), turned to 180 degrees
- moved C3 46.1 mm to (119.3, 76.9), turned to 180 degrees
- moved C9 46.0 mm to (122.0, 72.5), turned to -90 degrees
- moved C8 46.0 mm to (122.0, 70.7), turned to -90 degrees
- moved C15 45.7 mm to (124.2, 79.0), turned to 180 degrees
- moved C16 45.6 mm to (124.2, 79.9), turned to 180 degrees
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Connections:
- D17 pad 2: VBUS_A -> A_VBUS
- D18 pad 2: VBUS_B -> B_VBUS
- R1 pad 2: Net-(J1-CC) -> Net-(J2-CC1)
- R2 pad 2: Net-(J1-D+) -> Net-(J2-DA-)
- R3 pad 2: Net-(J1-D-) -> Net-(J2-DA+)
- R5 pad 2: Net-(R5-Pad2) -> Net-(J1-Pin_1)
- U1 pad 17: unconnected-(U1-GPIO17-Pad17) -> DET
- U1 pad 18: unconnected-(U1-GPIO18-Pad18) -> CMD
- U1 pad 19: unconnected-(U1-GPIO19-Pad19) -> CLK
- U1 pad 20: unconnected-(U1-GPIO20-Pad20) -> DAT0
- U1 pad 21: unconnected-(U1-GPIO21-Pad21) -> DAT1
- U1 pad 22: unconnected-(U1-GPIO22-Pad22) -> DAT2
- U1 pad 23: unconnected-(U1-GPIO23-Pad23) -> DAT3
- U1 pad 33: Net-(J2-Pin_3) -> Net-(J4-Pin_3)
- U1 pad 34: Net-(J2-Pin_1) -> Net-(J4-Pin_1)
- U1 pad 42: DET -> unconnected-(U1-GPIO33-Pad42)
- U1 pad 43: CMD -> unconnected-(U1-GPIO34-Pad43)
- U1 pad 44: CLK -> unconnected-(U1-GPIO35-Pad44)
- U1 pad 45: DAT0 -> unconnected-(U1-GPIO36-Pad45)
- U1 pad 46: DAT1 -> unconnected-(U1-GPIO37-Pad46)
- U1 pad 47: DAT2 -> unconnected-(U1-GPIO38-Pad47)
- U1 pad 48: DAT3 -> unconnected-(U1-GPIO39-Pad48)
Routing:
- net DET: track 0.00 -> 140.1 mm, vias 0 -> 17
- net +3.3V: track 0.00 -> 83.4 mm, vias 0 -> 9
- net Net-(U1-ADC_AVDD): track 0.00 -> 72.4 mm, vias 0 -> 10
- net +5V: track 0.00 -> 48.1 mm, vias 0 -> 7
- net 1.1V: track 0.00 -> 45.7 mm, vias 0 -> 9
- net CMD: track 0.00 -> 37.1 mm, vias 0 -> 7
- net Net-(U1-QSPI_SD0): track 0.00 -> 35.4 mm, vias 0 -> 2
- net Net-(U1-QSPI_SD1): track 0.00 -> 32.8 mm, vias 0 -> 6
- net Net-(U1-QSPI_SCLK): track 0.00 -> 31.9 mm, vias 0 -> 3
- net Net-(U1-QSPI_SD2): track 0.00 -> 31.9 mm, vias 0 -> 2
- net Net-(U1-~{QSPI_SS}): track 0.00 -> 28.8 mm, vias 0 -> 3
- net Net-(U1-QSPI_SD3): track 0.00 -> 28.3 mm, vias 0 -> 2
- net Net-(U1-VREG_AVDD): track 0.00 -> 23.9 mm, vias 0 -> 2
- net Net-(R7-Pad2): track 0.00 -> 19.9 mm, vias 0 -> 2
- net DAT2: track 0.00 -> 19.4 mm, vias 0 -> 5
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Other:
- board size 8.4 x 4.1 mm -> 15.7 x 40.1 mm
- copper layers 2 -> 4
- board text added: "GND"
- board text added: "PiKey"
- board text added: "QSPI_SS"
- board text added: "Reset"
- board text added: "SWCLK"
- board text added: "SWDIO"
- board text added: "Thenewtechguy"

Commit message: Monday 4th May update
Connections:
- J3 pad 3: CMD -> Net-(J3-CMD)
Other:
- outline, holes or cut-outs redrawn
